Commit message: Update dual_piper.urdf to replace .dae mesh files with .obj files for improved compatibility and performance.

File: assets/aloha_new_description/urdf/dual_piper.urdf (robot description, URDF)
Before this commit: robot dual_piper, 29 links, 28 joints
Links:
- link left_base_link: geometry collision mesh filename=package://aloha_new_description/meshes/base_link.STL; visual mesh filename=package://aloha_new_description/meshes/dark_dae/base_link.o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
- link left_camera_link: geometry collision box size=0.02505 0.09 0.025; visual mesh filename=package://realsense2_description/meshes/d435.obj
- link left_link1: geometry collision mesh filename=package://aloha_new_description/meshes/link1.STL; visual mesh filename=package://aloha_new_description/meshes/dark_dae/link1.obj
- link left_link2: geometry collision mesh filename=package://aloha_new_description/meshes/link2.STL; visual mesh filename=package://aloha_new_description/meshes/dark_dae/link2.obj
- link left_link3: geometry collision mesh filename=package://aloha_new_description/meshes/link3.STL; visual mesh filename=package://aloha_new_description/meshes/dark_dae/link3.obj
- link left_link4: geometry collision mesh filename=package://aloha_new_description/meshes/link4.STL; visual mesh filename=package://aloha_new_description/meshes/dark_dae/link4.obj
- link left_link5: geometry collision mesh filename=package://aloha_new_description/meshes/link5.STL; visual mesh filename=package://aloha_new_description/meshes/dark_dae/link5.obj
- link left_link6: geometry collision mesh filename=package://aloha_new_description/meshes/piper_slave_meshes/l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; visual mesh filename=package://aloha_new_description/meshes/dark_dae/link6_.obj
- link left_link7: geometry collision mesh filename=package://aloha_new_description/meshes/piper_slave_meshes/l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; visual mesh filename=package://aloha_new_description/meshes/dark_dae/link7.obj
- link left_link8: geometry collision mesh filename=package://aloha_new_description/meshes/piper_slave_meshes/l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; visual mesh filename=package://aloha_new_description/meshes/dark_dae/link8.obj
- link right_base_link: geometry collision mesh filename=package://aloha_new_description/meshes/base_link.STL; visual mesh filename=package://aloha_new_description/meshes/dark_dae/base_link.o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
- link right_camera_link: geometry collision box size=0.02505 0.09 0.025; visual mesh filename=package://realsense2_description/meshes/d435.obj
- link right_link1: geometry collision mesh filename=package://aloha_new_description/meshes/link1.STL; visual mesh filename=package://aloha_new_description/meshes/dark_dae/link1.obj
- link right_link2: geometry collision mesh filename=package://aloha_new_description/meshes/link2.STL; visual mesh filename=package://aloha_new_description/meshes/dark_dae/link2.obj
- link right_link3: geometry collision mesh filename=package://aloha_new_description/meshes/link3.STL; visual mesh filename=package://aloha_new_description/meshes/dark_dae/link3.obj
- link right_link4: geometry collision mesh filename=package://aloha_new_description/meshes/link4.STL; visual mesh filename=package://aloha_new_description/meshes/dark_dae/link4.obj
- link right_link5: geometry collision mesh filename=package://aloha_new_description/meshes/link5.STL; visual mesh filename=package://aloha_new_description/meshes/dark_dae/link5.obj
- link right_link6: geometry collision mesh filename=package://aloha_new_description/meshes/piper_slave_meshes/l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; visual mesh filename=package://aloha_new_description/meshes/dark_dae/link6_.obj
- link right_link7: geometry collision mesh filename=package://aloha_new_description/meshes/piper_slave_meshes/l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; visual mesh filename=package://aloha_new_description/meshes/dark_dae/link7.obj
- link right_link8: geometry collision mesh filename=package://aloha_new_description/meshes/piper_slave_meshes/l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; visual mesh filename=package://aloha_new_description/meshes/dark_dae/link8.obj
