Commit message: Update joint limits in dual_piper.urdf to use full range of motion, modify IK script to point to new JSON path, and enhance rendering options. Adjust camera matrix handling in isaac_sim_env.py for improved clarity and performance.

File: assets/aloha_new_description/urdf/dual_piper_origin.urdf (robot description, URDF)
Before this commit: robot dual_piper, 29 links, 28 joints
Joints:
- joint left_joint1: limit lower=-3.14159 upper=3.14159 effort=100 velocity=3 -> lower=-2.618 upper=2.618 effort=100 velocity=3
- joint left_joint2: limit lower=-3.14159 upper=3.14159 effort=100 velocity=3 -> lower=0 upper=3.14 effort=100 velocity=3
- joint left_joint3: limit lower=-3.14159 upper=3.14159 effort=100 velocity=3 -> lower=-2.697 upper=0 effort=100 velocity=3
- joint left_joint4: limit lower=-3.14159 upper=3.14159 effort=100 velocity=3 -> lower=-1.832 upper=1.832 effort=100 velocity=3
- joint left_joint5: limit lower=-3.14159 upper=3.14159 effort=100 velocity=3 -> lower=-1.22 upper=1.22 effort=100 velocity=3
- joint left_joint6: limit lower=-3.14159 upper=3.14159 effort=100 velocity=3 -> lower=-3.14 upper=3.14 effort=100 velocity=3
- joint right_joint1: limit lower=-3.14159 upper=3.14159 effort=100 velocity=3 -> lower=-2.618 upper=2.618 effort=100 velocity=3
- joint right_joint2: limit lower=-3.14159 upper=3.14159 effort=100 velocity=3 -> lower=0 upper=3.14 effort=100 velocity=3
- joint right_joint3: limit lower=-3.14159 upper=3.14159 effort=100 velocity=3 -> lower=-2.697 upper=0 effort=100 velocity=3
- joint right_joint4: limit lower=-3.14159 upper=3.14159 effort=100 velocity=3 -> lower=-1.832 upper=1.832 effort=100 velocity=3
- joint right_joint5: limit lower=-3.14159 upper=3.14159 effort=100 velocity=3 -> lower=-1.22 upper=1.22 effort=100 velocity=3
- joint right_joint6: limit lower=-3.14159 upper=3.14159 effort=100 velocity=3 -> lower=-3.14 upper=3.14 effort=100 velocity=3
